File: analog-led/analog-led/analog-led.kicad_pcb (KiCad board)
At the start: 2 copper layers, 51 parts, among them Q1 BC547, Q2 BC547, Q3 BC547, Q4 BC547

Commit message: Improved layout and schematic
Parts:
- added C10: C_Small, Capacitor_SMD:C_0603_1608Metric, F.Cu at (78.9, 27.9)
- added C11: C_Small, Capacitor_SMD:C_0603_1608Metric, F.Cu at (111.1, 31.6)
- added C8: C_Small, Capacitor_SMD:C_0603_1608Metric, F.Cu at (78.5, 34.2)
- added C9: C_Small, Capacitor_SMD:C_0603_1608Metric, F.Cu at (80.4, 20.4)
- added D33: LED, Diode_SMD:D_0603_1608Metric, F.Cu at (106.3, 91.5)
- added D34: LED, Diode_SMD:D_0603_1608Metric, F.Cu at (110.7, 91.5)
- added D35: LED, Diode_SMD:D_0603_1608Metric, F.Cu at (59.3, 20.3)
- added D36: LED, Diode_SMD:D_0603_1608Metric, F.Cu at (57.4, 27.9)
- added D37: LED, Diode_SMD:D_0603_1608Metric, F.Cu at (93.6, 31.6)
- added D38: LED, Diode_SMD:D_0603_1608Metric, F.Cu at (86.6, 51.8)
- added D39: LED, Diode_SMD:D_0603_1608Metric, F.Cu at (113.3, 22.9)
- added D40: LED, Diode_SMD:D_0603_1608Metric, F.Cu at (85.3, 41.7)
- added D41: LED, Diode_SMD:D_0603_1608Metric, F.Cu at (95.5, 22.9)
- added D42: LED, Diode_SMD:D_0603_1608Metric, F.Cu at (106.9, 31.6)
- added D43: LED, Diode_SMD:D_0603_1608Metric, F.Cu at (95.5, 51.8)
- added D44: LED, Diode_SMD:D_0603_1608Metric, F.Cu at (115.2, 91.5)
- added D45: LED, Diode_SMD:D_0603_1608Metric, F.Cu at (61.8, 34.2)
- added D46: LED, Diode_SMD:D_0603_1608Metric, F.Cu at (94.2, 41.7)
- added D47: LED, Diode_SMD:D_0603_1608Metric, F.Cu at (51.6, 48.0)
- added D48: LED, Diode_SMD:D_0603_1608Metric, F.Cu at (122.2, 22.9)
- added D49: LED, Diode_SMD:D_1206_3216Metric, F.Cu at (102.5, 31.6)
- added D50: LED, Diode_SMD:D_0603_1608Metric, F.Cu at (66.3, 27.9)
- added D51: LED, Diode_SMD:D_0603_1608Metric, F.Cu at (97.4, 91.5)
- added D52: LED, Diode_SMD:D_0603_1608Metric, F.Cu at (119.6, 91.5)
- added D53: LED, Diode_SMD:D_0603_1608Metric, F.Cu at (66.3, 34.2)
- added D54: LED, Diode_SMD:D_0603_1608Metric, F.Cu at (98.7, 41.7)
- added D55: LED, Diode_SMD:D_0603_1608Metric, F.Cu at (56.1, 48.0)
- added D56: LED, Diode_SMD:D_0603_1608Metric, F.Cu at (126.6, 22.9)
- added D57: LED, Diode_SMD:D_0603_1608Metric, F.Cu at (99.9, 51.8)
- added D58: LED, Diode_SMD:D_0603_1608Metric, F.Cu at (70.7, 27.9)
- added D59: LED, Diode_SMD:D_0603_1608Metric, F.Cu at (63.7, 20.3)
- added D60: LED, Diode_SMD:D_0603_1608Metric, F.Cu at (68.2, 20.3)
- added D61: LED, Diode_SMD:D_0603_1608Metric, F.Cu at (52.9, 34.2)
- added D62: LED, Diode_SMD:D_0603_1608Metric, F.Cu at (45.9, 20.3)
- added D63: LED, Diode_SMD:D_0603_1608Metric, F.Cu at (99.9, 22.9)
- added D64: LED, Diode_SMD:D_0603_1608Metric, F.Cu at (92.9, 91.5)
- added D65: D_Zener, Diode_SMD:D_0603_1608Metric, F.Cu at (21.7, 64.8)
- added F1: Fuse, Fuse:Fuse_1206_3216Metric, F.Cu at (26.7, 66.0)
- added J1: USB_B_Micro, Connector_USB:USB_Micro-B_GCT_USB3076-30-A, F.Cu at (103.0, 101.7)
- added Q5: BC547, Package_TO_SOT_SMD:SOT-23, F.Cu at (136.5, 45.7)
- added Q6: BC547, Package_TO_SOT_SMD:SOT-23, F.Cu at (144.8, 52.1)
- added Q7: BC547, Package_TO_SOT_SMD:SOT-23, F.Cu at (132.1, 45.7)
- added Q8: BC547, Package_TO_SOT_SMD:SOT-23, F.Cu at (132.1, 50.3)
- added R10: R_Small_US, Resistor_SMD:R_0603_1608Metric, F.Cu at (74.9, 27.9)
- added R11: R_Small_US, Resistor_SMD:R_0603_1608Metric, F.Cu at (76.4, 20.3)
- added R12: R_Small_US, Resistor_SMD:R_0603_1608Metric, F.Cu at (74.5, 34.2)
- added R13: R_Small_US, Resistor_SMD:R_0603_1608Metric, F.Cu at (106.9, 41.8)
- added R14: 22K, Resistor_SMD:R_0603_1608Metric, F.Cu at (102.9, 41.7)
- added R15: R_Small_US, Resistor_SMD:R_0603_1608Metric, F.Cu at (64.3, 48.0)
- added R16: R_Small_US, Resistor_SMD:R_0603_1608Metric, F.Cu at (108.1, 51.9)
- added R9: R_Small_US, Resistor_SMD:R_0603_1608Metric, F.Cu at (104.1, 51.8)
- added U1: AZ1117-3.3, Package_TO_SOT_SMD:SOT-223, F.Cu at (26.7, 58.4)
- D1, D10, D11, D12, D13, D14, D15, D16, D17, D18, D19, D2, D20, D21, D22, D23, D24, D25, D26, D27, D28, D29, D3, D30, D31, D32, D4, D5, D6, D7, D8, D9: footprint Diode_SMD:D_0603_1608Metric_Castellated -> Diode_SMD:D_0603_1608Metric
- Q1, Q2, Q3, Q4: footprint Package_TO_SOT_THT:TO-92_Inline -> Package_TO_SOT_SMD:SOT-23
- moved Q1 80.1 mm to (17.9, 84.3)
- moved Q2 77.1 mm to (17.9, 79.7)
- moved C5 70.2 mm to (127.8, 91.5)
- moved D14 69.6 mm to (21.8, 90.4)
- moved D10 69.5 mm to (21.8, 87.8)
- moved D4 69.2 mm to (17.7, 87.8)
- moved C6 68.6 mm to (123.8, 91.5)
- moved R7 65.1 mm to (130.8, 23.0)
- moved D7 64.5 mm to (17.7, 90.4)
- moved D29 63.6 mm to (117.7, 22.9)
- moved C2 63.3 mm to (29.8, 86.5)
- moved D1 62.6 mm to (25.8, 89.1)
- moved D21 60.1 mm to (101.8, 91.5)
- moved R3 59.7 mm to (29.8, 89.0)
- moved D9 57.9 mm to (22.2, 83.9)
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Connections:
- C3 pad 1: GND -> Net-(C3-Pad1)
- C3 pad 2: +3V3 -> Net-(C3-Pad2)
- C4 pad 1: GND -> Net-(C4-Pad1)
- C4 pad 2: +3V3 -> Net-(C4-Pad2)
- C5 pad 1: GND -> Net-(C5-Pad1)
- D10 pad 1: Net-(C6-Pad1) -> Net-(C2-Pad1)
- D11 pad 1: Net-(C6-Pad1) -> Net-(C2-Pad1)
- D12 pad 1: Net-(C6-Pad1) -> Net-(C2-Pad1)
- D13 pad 1: Net-(C6-Pad1) -> Net-(C2-Pad1)
- D14 pad 1: Net-(C6-Pad1) -> Net-(C2-Pad1)
- D15 pad 1: Net-(C6-Pad1) -> Net-(C2-Pad1)
- D16 pad 1: Net-(C6-Pad1) -> Net-(C2-Pad1)
- D17 pad 1: Net-(C7-Pad1) -> Net-(C3-Pad1)
- D18 pad 1: Net-(C7-Pad1) -> Net-(C3-Pad1)
- D19 pad 1: Net-(C7-Pad1) -> Net-(C3-Pad1)
- D20 pad 1: Net-(C7-Pad1) -> Net-(C3-Pad1)
- D21 pad 1: Net-(C7-Pad1) -> Net-(C3-Pad1)
- D22 pad 1: Net-(C7-Pad1) -> Net-(C3-Pad1)
- D23 pad 1: Net-(C7-Pad1) -> Net-(C3-Pad1)
- D24 pad 1: Net-(C7-Pad1) -> Net-(C3-Pad1)
- D25 pad 1: Net-(C1-Pad1) -> Net-(C4-Pad1)
- D25 pad 2: Net-(D1-Pad2) -> Net-(D25-Pad2)
- D26 pad 1: Net-(C1-Pad1) -> Net-(C4-Pad1)
- D26 pad 2: Net-(D1-Pad2) -> Net-(D25-Pad2)
- D27 pad 1: Net-(C1-Pad1) -> Net-(C4-Pad1)
- D27 pad 2: Net-(D1-Pad2) -> Net-(D25-Pad2)
- D28 pad 1: Net-(C1-Pad1) -> Net-(C4-Pad1)
- D28 pad 2: Net-(D1-Pad2) -> Net-(D25-Pad2)
- D29 pad 1: Net-(C2-Pad1) -> Net-(C4-Pad1)
- D29 pad 2: Net-(D29-Pad2) -> Net-(D25-Pad2)
- D30 pad 1: Net-(C2-Pad1) -> Net-(C4-Pad1)
- D30 pad 2: Net-(D29-Pad2) -> Net-(D25-Pad2)
- D31 pad 1: Net-(C2-Pad1) -> Net-(C4-Pad1)
- D31 pad 2: Net-(D29-Pad2) -> Net-(D25-Pad2)
- D32 pad 1: Net-(C2-Pad1) -> Net-(C4-Pad1)
- D32 pad 2: Net-(D29-Pad2) -> Net-(D25-Pad2)
- D5 pad 1: Net-(C2-Pad1) -> Net-(C1-Pad1)
- D5 pad 2: Net-(D29-Pad2) -> Net-(D1-Pad2)
- D6 pad 1: Net-(C2-Pad1) -> Net-(C1-Pad1)
- D6 pad 2: Net-(D29-Pad2) -> Net-(D1-Pad2)
- D7 pad 1: Net-(C2-Pad1) -> Net-(C1-Pad1)
- D7 pad 2: Net-(D29-Pad2) -> Net-(D1-Pad2)
- D8 pad 1: Net-(C2-Pad1) -> Net-(C1-Pad1)
- D8 pad 2: Net-(D29-Pad2) -> Net-(D1-Pad2)
- D9 pad 1: Net-(C6-Pad1) -> Net-(C2-Pad1)
- Q1 pad 2: Net-(C7-Pad2) -> +3V3
- Q3 pad 1: Net-(C6-Pad1) -> Net-(C3-Pad1)
- Q3 pad 2: +3V3 -> Net-(C2-Pad2)
- Q4 pad 1: Net-(C7-Pad1) -> Net-(C4-Pad1)
- Q4 pad 2: Net-(C6-Pad2) -> Net-(C3-Pad2)
- R3 pad 2: Net-(D29-Pad2) -> Net-(D10-Pad2)
- R5 pad 2: Net-(D10-Pad2) -> Net-(D17-Pad2)
- R6 pad 2: Net-(C6-Pad2) -> Net-(C3-Pad2)
- R7 pad 2: Net-(D17-Pad2) -> Net-(D25-Pad2)
- R8 pad 2: Net-(C7-Pad2) -> Net-(C4-Pad2)
