File: led-matrix/led-matrix/led-matrix.kicad_pcb (KiCad board)
At the start: 2 copper layers, 105.4 x 101.6 mm, 304 parts, among them J1 Conn_2Rows-05Pins, J2 Conn_2Rows-05Pins, J3 USB_B_Micro, Q1 2N7002, Q10 2N7002, Q11 2N7002, Q12 2N7002, Q13 2N7002, Q14 2N7002, Q15 2N7002, Q16 2N7002, Q2 2N7002, Q3 2N7002, Q4 2N7002, Q5 2N7002, Q6 2N7002, Q7 2N7002, Q8 2N7002, Q9 2N7002, U1 74LS595, U2 74LS595, U3 74LS595, U4 74LS595, U5 AMS1117-3.3

Commit message: Changes
Parts:
- J1, J2: moved to F.Cu
- J3: footprint Connector_USB:USB_Micro-B_Molex-105017-0001 -> Connector_USB:USB_Micro-B_Molex_47346-0001
- moved J1 126.8 mm to (26.7, 82.5)
- moved C1 26.8 mm to (64.8, 109.2), turned to 180 degrees
- moved J2 26.5 mm to (32.5, 82.5), turned to 0 degrees
- moved C4 14.3 mm to (64.8, 71.1), turned to 180 degrees
- moved C3 14.1 mm to (119.4, 129.5), turned to 270 degrees
- moved U1 13.1 mm to (64.7, 116.2), turned to 180 degrees
- moved C2 9.29 mm to (83.8, 129.1), turned to 270 degrees
- moved U3 8.89 mm to (77.5, 129.5)
- moved U2 5.23 mm to (64.8, 77.5), turned to 180 degrees
- moved C6 1.03 mm to (105.9, 81.6)
Routing:
- net GND: track 0.00 -> 296.5 mm, vias 0 -> 1
- net Net-(D110-Pad1): track 0.00 -> 132.6 mm, vias 0 -> 19
- net Net-(D111-Pad1): track 0.00 -> 131.8 mm, vias 0 -> 19
- net Net-(D114-Pad1): track 0.00 -> 128.4 mm, vias 0 -> 18
- net Net-(D109-Pad1): track 0.00 -> 127.3 mm, vias 0 -> 20
- net Net-(D115-Pad1): track 0.00 -> 127.1 mm, vias 0 -> 21
- net Net-(D100-Pad1): track 0.00 -> 125.1 mm, vias 0 -> 29
- net Net-(D101-Pad1): track 0.00 -> 122.4 mm, vias 0 -> 20
- net Net-(D108-Pad1): track 0.00 -> 121.3 mm, vias 0 -> 18
- net Net-(D112-Pad1): track 0.00 -> 119.8 mm, vias 0 -> 16
- net Net-(D1-Pad1): track 9.91 -> 129.6 mm, vias 2 -> 16
- net Net-(D102-Pad1): track 0.00 -> 118.4 mm, vias 0 -> 19
- net Net-(D103-Pad1): track 0.00 -> 112.9 mm, vias 0 -> 17
- net Net-(D107-Pad1): track 0.00 -> 110.6 mm, vias 0 -> 17
- net Net-(D10-Pad1): track 0.00 -> 101.3 mm, vias 0 -> 17
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Other:
- net class Default: clearance 0.2 -> 0.127; trace_width 0.25 -> 0.127; via_dia 0.8 -> 0.6; via_drill 0.4 -> 0.3
- rule pad_to_mask_clearance: 0.051 -> 0
- rule solder_mask_min_width: 0.25 -> 0.12
- rule trace_clearance: 0.2 -> 0.127
- rule trace_min: 0.2 -> 0.127
- rule via_min_size: 0.4 -> 0.6
