File: game-console/gameConsole/gameConsole.kicad_pcb (KiCad board)
At the start: 2 copper layers, 11 parts, among them U1 STM32F038C6Tx, U10 MPU-6050, U2 AD1855, U2 MCP4725xxx-xCH, U3 CS43L21, U3 DS1307Z+, U4 CS43L21, U5 STM32F100C8Tx, U7 MCP4725xxx-xCH, U9 AP1117-33

Commit message: Added init kicad source files
Parts:
- removed U1: STM32F038C6Tx, Package_QFP:LQFP-48_7x7mm_P0.5mm
- added U4: RP2040, Package_DFN_QFN:QFN-56-1EP_7x7mm_P0.4mm_EP3.2x3.2mm, F.Cu at (161.7, 64.3)
- U5: value STM32F100C8Tx -> RP2040; footprint Package_QFP:LQFP-48_7x7mm_P0.5mm -> Package_DFN_QFN:QFN-56-1EP_7x7mm_P0.4mm_EP3.2x3.2mm
- moved U5 12.7 mm to (161.7, 73.6)
Connections:
- net +3V3 renamed +3.3V
- DS1 pad 1: Net-(DS1-Pad1) -> unconnected-(DS1-VCC-Pad1)
- DS1 pad 10: Net-(DS1-Pad10) -> unconnected-(DS1-DB6-Pad10)
- DS1 pad 11: Net-(DS1-Pad11) -> unconnected-(DS1-DB7-Pad11)
- DS1 pad 12: Net-(DS1-Pad12) -> unconnected-(DS1-~{CS1}-Pad12)
- DS1 pad 13: Net-(DS1-Pad13) -> unconnected-(DS1-~{CS2}-Pad13)
- DS1 pad 14: Net-(DS1-Pad14) -> unconnected-(DS1-~{RST}-Pad14)
- DS1 pad 15: Net-(DS1-Pad15) -> unconnected-(DS1-R/~{W}-Pad15)
- DS1 pad 16: Net-(DS1-Pad16) -> unconnected-(DS1-D/~{I}-Pad16)
- DS1 pad 17: Net-(DS1-Pad17) -> unconnected-(DS1-E-Pad17)
- DS1 pad 18: Net-(DS1-Pad18) -> unconnected-(DS1-VEE-Pad18)
- DS1 pad 19: Net-(DS1-Pad19) -> unconnected-(DS1-LEDA/EL-Pad19)
- DS1 pad 2: Net-(DS1-Pad2) -> unconnected-(DS1-GND-Pad2)
- DS1 pad 20: Net-(DS1-Pad20) -> unconnected-(DS1-LEDK/EL-Pad20)
- DS1 pad 3: Net-(DS1-Pad3) -> unconnected-(DS1-VO-Pad3)
- DS1 pad 4: Net-(DS1-Pad4) -> unconnected-(DS1-DB0-Pad4)
- DS1 pad 5: Net-(DS1-Pad5) -> unconnected-(DS1-DB1-Pad5)
- DS1 pad 6: Net-(DS1-Pad6) -> unconnected-(DS1-DB2-Pad6)
- DS1 pad 7: Net-(DS1-Pad7) -> unconnected-(DS1-DB3-Pad7)
- DS1 pad 8: Net-(DS1-Pad8) -> unconnected-(DS1-DB4-Pad8)
- DS1 pad 9: Net-(DS1-Pad9) -> unconnected-(DS1-DB5-Pad9)
- U10 pad 1: Net-(U10-Pad1) -> unconnected-(U10-CLKIN-Pad1)
- U10 pad 10: Net-(U10-Pad10) -> unconnected-(U10-REGOUT-Pad10)
- U10 pad 11: Net-(U10-Pad11) -> unconnected-(U10-FSYNC-Pad11)
- U10 pad 12: Net-(U10-Pad12) -> unconnected-(U10-INT-Pad12)
- U10 pad 14: (no net) -> unconnected-(U10-NC-Pad14)
- U10 pad 15: (no net) -> unconnected-(U10-NC-Pad15)
- U10 pad 16: (no net) -> unconnected-(U10-NC-Pad16)
- U10 pad 17: (no net) -> unconnected-(U10-NC-Pad17)
- U10 pad 19: (no net) -> unconnected-(U10-RESV-Pad19)
- U10 pad 2: (no net) -> unconnected-(U10-NC-Pad2)
- U10 pad 20: Net-(U10-Pad20) -> unconnected-(U10-CPOUT-Pad20)
- U10 pad 21: (no net) -> unconnected-(U10-RESV-Pad21)
- U10 pad 22: (no net) -> unconnected-(U10-RESV-Pad22)
- U10 pad 3: (no net) -> unconnected-(U10-NC-Pad3)
- U10 pad 4: (no net) -> unconnected-(U10-NC-Pad4)
- U10 pad 5: (no net) -> unconnected-(U10-NC-Pad5)
- U10 pad 6: Net-(U10-Pad6) -> unconnected-(U10-AUX_DA-Pad6)
- U10 pad 7: Net-(U10-Pad7) -> unconnected-(U10-AUX_CL-Pad7)
- U10 pad 8: Net-(U10-Pad8) -> unconnected-(U10-VLOGIC-Pad8)
- U10 pad 9: Net-(U10-Pad9) -> unconnected-(U10-AD0-Pad9)
- U3 pad 1: Net-(U3-Pad1) -> Net-(U3-X1)
- U3 pad 2: Net-(U3-Pad2) -> Net-(U3-X2)
- U3 pad 3: Net-(U3-Pad3) -> unconnected-(U3-VBAT-Pad3)
- U3 pad 7: Net-(U3-Pad7) -> unconnected-(U3-SQW/OUT-Pad7)
- U5 pad 1: Net-(U5-Pad1) -> Net-(U5-IOVDD-Pad1)
- U5 pad 10: Net-(U5-Pad10) -> Net-(U5-IOVDD-Pad1)
- U5 pad 11: Net-(U5-Pad11) -> unconnected-(U5-GPIO8-Pad11)
- U5 pad 12: Net-(U5-Pad12) -> unconnected-(U5-GPIO9-Pad12)
- U5 pad 13: Net-(U5-Pad13) -> unconnected-(U5-GPIO10-Pad13)
- U5 pad 14: Net-(U5-Pad14) -> unconnected-(U5-GPIO11-Pad14)
- U5 pad 15: Net-(U5-Pad15) -> unconnected-(U5-GPIO12-Pad15)
- U5 pad 16: Net-(U5-Pad16) -> unconnected-(U5-GPIO13-Pad16)
- U5 pad 17: Net-(U5-Pad17) -> unconnected-(U5-GPIO14-Pad17)
- U5 pad 18: Net-(U5-Pad18) -> unconnected-(U5-GPIO15-Pad18)
- U5 pad 19: Net-(U5-Pad19) -> unconnected-(U5-TESTEN-Pad19)
- U5 pad 2: Net-(U5-Pad2) -> unconnected-(U5-GPIO0-Pad2)
- U5 pad 20: Net-(U5-Pad20) -> unconnected-(U5-XIN-Pad20)
- U5 pad 21: Net-(U5-Pad21) -> unconnected-(U5-XOUT-Pad21)
- U5 pad 22: Net-(U5-Pad22) -> Net-(U5-IOVDD-Pad1)
- U5 pad 23: Net-(U5-Pad23) -> Net-(U5-DVDD-Pad23)
- U5 pad 24: Net-(U5-Pad24) -> unconnected-(U5-SWCLK-Pad24)
- U5 pad 25: Net-(U5-Pad25) -> unconnected-(U5-SWD-Pad25)
- U5 pad 26: Net-(U5-Pad26) -> unconnected-(U5-RUN-Pad26)
- U5 pad 27: Net-(U5-Pad27) -> unconnected-(U5-GPIO16-Pad27)
- U5 pad 28: Net-(U5-Pad28) -> unconnected-(U5-GPIO17-Pad28)
- U5 pad 29: Net-(U5-Pad29) -> unconnected-(U5-GPIO18-Pad29)
- U5 pad 3: Net-(U5-Pad3) -> unconnected-(U5-GPIO1-Pad3)
- U5 pad 30: Net-(U5-Pad30) -> unconnected-(U5-GPIO19-Pad30)
- U5 pad 31: Net-(U5-Pad31) -> unconnected-(U5-GPIO20-Pad31)
- U5 pad 32: Net-(U5-Pad32) -> unconnected-(U5-GPIO21-Pad32)
- U5 pad 33: Net-(U5-Pad33) -> Net-(U5-IOVDD-Pad1)
- U5 pad 34: Net-(U5-Pad34) -> unconnected-(U5-GPIO22-Pad34)
- U5 pad 35: Net-(U5-Pad35) -> unconnected-(U5-GPIO23-Pad35)
- U5 pad 36: Net-(U5-Pad36) -> unconnected-(U5-GPIO24-Pad36)
- U5 pad 37: Net-(U5-Pad37) -> unconnected-(U5-GPIO25-Pad37)
- U5 pad 38: Net-(U5-Pad38) -> unconnected-(U5-GPIO26_ADC0-Pad38)
- U5 pad 39: Net-(U5-Pad39) -> unconnected-(U5-GPIO27_ADC1-Pad39)
- U5 pad 4: Net-(U5-Pad4) -> unconnected-(U5-GPIO2-Pad4)
- U5 pad 40: Net-(U5-Pad40) -> unconnected-(U5-GPIO28_ADC2-Pad40)
- U5 pad 41: Net-(U5-Pad41) -> unconnected-(U5-GPIO29_ADC3-Pad41)
- U5 pad 42: Net-(U5-Pad42) -> Net-(U5-IOVDD-Pad1)
- U5 pad 43: Net-(U5-Pad43) -> unconnected-(U5-ADC_AVDD-Pad43)
- U5 pad 44: Net-(U5-Pad44) -> unconnected-(U5-VREG_IN-Pad44)
- U5 pad 45: Net-(U5-Pad45) -> unconnected-(U5-VREG_VOUT-Pad45)
- U5 pad 46: Net-(U5-Pad46) -> unconnected-(U5-USB_DM-Pad46)
- U5 pad 47: Net-(U5-Pad47) -> unconnected-(U5-USB_DP-Pad47)
- U5 pad 48: Net-(U5-Pad48) -> unconnected-(U5-USB_VDD-Pad48)
- U5 pad 5: Net-(U5-Pad5) -> unconnected-(U5-GPIO3-Pad5)
- U5 pad 6: Net-(U5-Pad6) -> unconnected-(U5-GPIO4-Pad6)
- U5 pad 7: Net-(U5-Pad7) -> unconnected-(U5-GPIO5-Pad7)
- U5 pad 8: Net-(U5-Pad8) -> unconnected-(U5-GPIO6-Pad8)
- U5 pad 9: Net-(U5-Pad9) -> unconnected-(U5-GPIO7-Pad9)
- U9 pad 1: Net-(U9-Pad1) -> unconnected-(U9-GND-Pad1)
- U9 pad 2: Net-(U9-Pad2) -> unconnected-(U9-VO-Pad2)
- U9 pad 3: Net-(U9-Pad3) -> unconnected-(U9-VI-Pad3)
Other:
- net class Default removed

Commit message: Minor improvements
Parts:
- moved U2 27.7 mm to (98.0, 25.1)
Changed lines of the file:
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@@
   (net 249 "unconnected-(U10-CLKIN-Pad1)")
   (footprint "Package_SO:SSOP-28_5.3x10.2mm_P0.65mm" (layer "F.Cu")
-    (at 87.63 50.8)
+    (at 98 25.075)
     (descr "28-Lead Plastic Shrink Small Outline (SS)-5.30 mm Body [SSOP] (see Microchip Packaging Specification 00000049BS.pdf)")
     (tags "SSOP 0.65")
