File: game-console/gameConsole/gameConsole.kicad_sch (KiCad schematic)
At the start: 51 parts, among them J1 Micro_SD_Card, J2 AudioJack2_Switch, J3 USB_B_Micro, SW1 SW_Push, U1 24LC1025, U10 MPU-6050, U11 PAM8403, U2 MCP4725xxx-xCH, U3 DS1307Z+, U4 RP2040, U5 RP2040, U7 MCP4725xxx-xCH, U9 AP1117-33, Y1 Crystal, Y2 Crystal

Commit message: Minor improvements
Parts:
- added C1, C24, C25: C, symbol pspice:C
- added P1: USB_C_Plug, symbol Connector:USB_C_Plug
- added R12, R13, R14, R15: 27R, symbol Device:R_US
- added U6: W25Q32JVSS, Package_SO:SOIC-8_5.23x5.23mm_P1.27mm, symbol Memory_Flash:W25Q32JVSS
Connections:
- net +3.3V: now also J1.4 (VDD), U4.1 (IOVDD), U4.10 (IOVDD), U4.22 (IOVDD), U4.33 (IOVDD), U4.42 (IOVDD), U4.49 (IOVDD)
- net +5V: now also P1.A4 (VBUS), P1.A9 (VBUS), P1.B4 (VBUS), P1.B9 (VBUS)
- net GND: now also J1.6 (VSS), P1.A1 (GND), P1.A12 (GND), P1.B1 (GND), P1.B12 (GND)
- net QSPI_SCLK: now reaches J1.5 (CLK)
- net QSPI_SCLK: now also U4.52 (QSPI_SCLK)
- net at Y1.1: now also C24.2, R14.1
- net at Y1.2: now also C25.2, R15.2
- net CPU0SPI0TX: now reaches U4.2 (GPIO0)
- net CPU0SPI0TX: now also U5.5 (GPIO3)
- net CPU0SPI0SCK: now reaches U4.4 (GPIO2)
- net CPU0SPI0SCK: now also U5.4 (GPIO2)
- net at U4.46 (USB_DM): now also R12.2
- net at U4.47 (USB_DP): now also R13.2
- net CPU0SPI0RX: now reaches U4.5 (GPIO3)
- net CPU0SPI0RX: now also U5.2 (GPIO0)
- net QSPI_SD0: now reaches U4.53 (QSPI_SD0)
- net QSPI_SD1: now reaches U4.55 (QSPI_SD1)
- net CPUQSPI_SS: now reaches U4.56 (QSPI_SS)
- new net: R14.2, R15.1
- new net USBD+: P1.A6 (D+), R13.1
- new net USBD-: P1.A7 (D-), R12.1
Other:
- moved on the sheet: C16, C2, J1, R1, R2, U3, U4, U5, Y1, Y2
