File: clock-matrix/schematic/clock-matrix.sch (EAGLE design)
At the start: 80 parts, among them IC1 WS2811-SOP8, IC2 WS2811-SOP8, IC3 74HC595D, U1 Tiny45-20-SMT, X2 USB-MICROB

Commit message: Relocated files, removed unused files, updated christmas and clock board and other changes
Parts:
- removed U1: Tiny45-20-SMT, SparkFun-Retired:ATTINY45TINY45-20-SMT
- added C6: (no value), rcl:C-EUC0603
- added R2, R4, R7, R8: 33, adafruit:R-US_R0603
- added U2: ATMEGA328P-MU, Microcontroller:ATMEGA328P-MU
- R3: value 0 -> 33; device audio amplifier example:R-US_R1206 -> adafruit:R-US_R0603
Connections:
- removed net CLK: IC3A.SCK, S1.1, U1.PB3(ADC3)
- removed net RCK: IC3A.RCK, U1.PB4(ADC2)
- new net BT0: R2.1, S2.1, U2.PD2(INT0/PCINT18)
- new net BT1: R3.1, S1.1, U2.PD3(PCINT19/OC2B/INT1)
- new net LATCH: C6.1, IC3A.RCK, U2.(ADC2/PCINT10)PC2
- new net LEDDATA: R9.1, U2.(PCINT0/CLKO/ICP1)PB0
- new net MISO: TP2.TP, U2.(PCINT4/MISO)PB4
- new net MOSI: TP3.TP, U2.(PCINT3/OC2A/MOSI)PB3
- new net N$13: IC2.SET, R8.2
- new net N$4: IC1.SET, R7.2
- new net N$6: U2.(PCINT7/XTAL2/TOSC2)PB7
- new net N$8: U2.(PCINT6/XTAL1/TOSC1)PB6
- new net PWM: IC3A.G, U2.(PCINT1/OC1A)PB1
- new net RCLK: IC3A.SCK, U2.(ADC1/PCINT9)PC1
- new net RX: U2.PD0(RXD/PCINT16)
- new net SCK: TP4.TP, U2.(SCK/PCINT5)PB5
- new net TX: U2.PD1(TXD/PCINT17)
- net 5V: now also R2.2, R3.2, R7.1, R8.1, U2.AVCC, U2.VCC, U2.VCC1; no longer S1.2, U1.VCC
- net GND: now also C6.2, S1.2, U2.GND, U2.GND1, U2.GND2; no longer IC3A.G, U1.GND
- net N$5: now also IC2.DO, R4.2; no longer IC3A.QH*, R3.1
- net RES: now also U2.(RESET/PCINT14)PC6; no longer R9.1, S2.1, U1.PB5(NRES)
- net SCL: now also U2.(ADC5/SCL/PCINT13)PC5; no longer TP3.TP, U1.PB2(SCK/ADC1)
- net SDA: now also U2.(ADC4/SDA/PCINT12)PC4; no longer TP4.TP, U1.PB0(MOSI)
- net SER: now also U2.(ADC3/PCINT11)PC3; no longer R3.2, TP2.TP, U1.PB1(MISO)
Other:
- moved on the sheet: BAT1, C1, C18, C2, C3, C4, C5, D2, F1, IC3, IC3P, LED1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

Commit message: Removed unused files, update board, code and other changes
Parts:
- TP1, TP2, TP3, TP4, TP5, TP6: value TPB1,27 -> TPTP10R; device testpad:TPB1,27 -> testpad:TPTP10R
Changed lines of the file:
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@@
 <part name="GND7" library="SparkFun" deviceset="GND" device=""/>
 <part name="X2" library="SparkFun" deviceset="USB" device="-MICROB"/>
-<part name="TP1" library="testpad" deviceset="TP" device="B1,27"/>
-<part name="TP2" library="testpad" deviceset="TP" device="B1,27"/>
-<part name="TP3" library="testpad" deviceset="TP" device="B1,27"/>
-<part name="TP5" library="testpad" deviceset="TP" device="B1,27"/>
-<part name="TP6" library="testpad" deviceset="TP" device="B1,27"/>
-<part name="TP4" library="testpad" deviceset="TP" device="B1,27"/>
+<part name="TP1" library="testpad" library_urn="urn:adsk.eagle:library:385" deviceset="TP" device="TP10R" package3d_urn="urn:adsk.eagle:package:27959/1"/>
+<part name="TP2" library="testpad" library_urn="urn:adsk.eagle:library:385" deviceset="TP" device="TP10R" package3d_urn="urn:adsk.eagle:package:27959/1"/>
+<part name="TP3" library="testpad" library_urn="urn:adsk.eagle:library:385" deviceset="TP" device="TP10R" package3d_urn="urn:adsk.eagle:package:27959/1"/>
+<part name="TP5" library="testpad" library_urn="urn:adsk.eagle:library:385" deviceset="TP" device="TP10R" package3d_urn="urn:adsk.eagle:package:27959/1"/>
+<part name="TP6" library="testpad" library_urn="urn:adsk.eagle:library:385" deviceset="TP" device="TP10R" package3d_urn="urn:adsk.eagle:package:27959/1" value="TPTP10R"/>
+<part name="TP4" library="testpad" library_urn="urn:adsk.eagle:library:385" deviceset="TP" device="TP10R" package3d_urn="urn:adsk.eagle:package:27959/1"/>
 <part name="LED13" library="SparkFun" deviceset="LED" device="1206"/>
 <part name="LED14" library="SparkFun" deviceset="LED" device="1206"/>

Commit message: Improvement and other changes
Parts:
- C3: value (none) -> 100nF
- C6: value (none) -> 10nF
Changed lines of the file:
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@@
 <part name="GND2" library="SparkFun" deviceset="GND" device=""/>
 <part name="U$11" library="SparkFun" deviceset="5V" device=""/>
-<part name="C3" library="rcl" deviceset="C-EU" device="C0603"/>
+<part name="C3" library="rcl" deviceset="C-EU" device="C0603" value="100nF"/>
 <part name="U$12" library="SparkFun" deviceset="5V" device=""/>
 <part name="U$13" library="SparkFun" deviceset="5V" device=""/>
@@
 <part name="R7" library="adafruit" deviceset="R-US_" device="R0603" value="33"/>
 <part name="R8" library="adafruit" deviceset="R-US_" device="R0603" value="33"/>
-<part name="C6" library="rcl" deviceset="C-EU" device="C0603"/>
+<part name="C6" library="rcl" deviceset="C-EU" device="C0603" value="10nF"/>
 <part name="GND3" library="SparkFun" deviceset="GND" device=""/>
 </parts>
