File: clock-matrix/schematic/clock-matrix.brd (EAGLE design)
At the start: 30 x 50 mm, 85 parts, among them IC1 WS2811-SOP8, IC2 WS2811-SOP8, IC3 74HC595D, U2 ATMEGA328P-MU, X2 USB-MICROB

Commit message: Removed unused files, update board, code and other changes
Parts:
- TP1, TP2, TP3, TP4, TP5, TP6: value TPB1,27 -> TPTP10R; device testpad:B1,27 -> testpad:TP10R
Changed lines of the file:
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@@
 <drawing>
 <settings>
-<setting alwaysvectorfont="yes"/>
+<setting alwaysvectorfont="no"/>
 <setting verticaltext="up"/>
 </settings>
 <grid distance="0.2" unitdist="mm" unit="mm" style="lines" multiple="1" display="no" altdistance="5" altunitdist="mil" altunit="mm"/>
 <layers>
-<layer number="1" name="Top" color="4" fill="1" visible="yes" active="yes"/>
+<layer number="1" name="Top" color="4" fill="1" visible="no" active="yes"/>
 <layer number="16" name="Bottom" color="1" fill="1" visible="yes" active="yes"/>
 <layer number="17" name="Pads" color="2" fill="1" visible="yes" active="yes"/>
@@
 <layer number="19" name="Unrouted" color="6" fill="1" visible="yes" active="yes"/>
 <layer number="20" name="Dimension" color="24" fill="1" visible="yes" active="yes"/>
-<layer number="21" name="tPlace" color="7" fill="1" visible="yes" active="yes"/>
+<layer number="21" name="tPlace" color="7" fill="1" visible="no" active="yes"/>
 <layer number="22" name="bPlace" color="7" fill="1" visible="yes" active="yes"/>
-<layer number="23" name="tOrigins" color="15" fill="1" visible="yes" active="yes"/>
+<layer number="23" name="tOrigins" color="15" fill="1" visible="no" active="yes"/>
 <layer number="24" name="bOrigins" color="15" fill="1" visible="yes" active="yes"/>
-<layer number="25" name="tNames" color="7" fill="1" visible="yes" active="yes"/>
+<layer number="25" name="tNames" color="7" fill="1" visible="no" active="yes"/>
 <layer number="26" name="bNames" color="7" fill="1" visible="yes" active="yes"/>
 <layer number="27" name="tValues" color="7" fill="1" visible="no" active="yes"/>
@@
 <layer number="37" name="tTest" color="7" fill="1" visible="no" active="yes"/>
 <layer number="38" name="bTest" color="7" fill="1" visible="no" active="yes"/>
-<layer number="39" name="tKeepout" color="4" fill="11" visible="yes" active="yes"/>
+<layer number="39" name="tKeepout" color="4" fill="11" visible="no" active="yes"/>
 <layer number="40" name="bKeepout" color="1" fill="11" visible="yes" active="yes"/>
-<layer number="41" name="tRestrict" color="4" fill="10" visible="yes" active="yes"/>
+<layer number="41" name="tRestrict" color="4" fill="10" visible="no" active="yes"/>
 <layer number="42" name="bRestrict" color="1" fill="10" visible="yes" active="yes"/>
 <layer number="43" name="vRestrict" color="2" fill="10" visible="no" active="yes"/>
@@
 <layer number="49" name="Reference" color="7" fill="1" visible="no" active="yes"/>
 <layer number="50" name="dxf" color="7" fill="1" visible="no" active="no"/>
-<layer number="51" name="tDocu" color="7" fill="1" visible="yes" active="yes"/>
+<layer number="51" name="tDocu" color="7" fill="1" visible="no" active="yes"/>
 <layer number="52" name="bDocu" color="7" fill="1" visible="yes" active="yes"/>
 <layer number="53" name="tGND_GNDA" color="7" fill="9" visible="no" active="no"/>
@@
 <attribute name="NAME" x="4.941" y="16.329" size="1.27" layer="26" rot="MR270"/>
 </element>
-<element name="TP1" library="testpad" package="B1,27" value="TPB1,27" x="10.43" y="26.1" smashed="yes" rot="MR0">
+<element name="TP1" library="testpad" library_urn="urn:adsk.eagle:library:385" package="TP10R" package3d_urn="urn:adsk.eagle:package:27959/1" value="TPTP10R" x="10.43" y="26.1" smashed="yes" rot="MR0">
+<attribute name="POPULARITY" value="3" x="10.43" y="26.1" size="1.778" layer="28" rot="MR0" display="off"/>
 <attribute name="TP_SIGNAL_NAME" value="" x="11.065" y="24.195" size="1" layer="38" rot="MR0"/>
 <attribute name="VALUE" x="11.065" y="25.338" size="0.0254" layer="28" rot="MR0"/>
 </element>
-<element name="TP2" library="testpad" package="B1,27" value="TPB1,27" x="2.91" y="30.25" smashed="yes" rot="MR0">
+<element name="TP2" library="testpad" library_urn="urn:adsk.eagle:library:385" package="TP10R" package3d_urn="urn:adsk.eagle:package:27959/1" value="TPTP10R" x="2.91" y="30.25" smashed="yes" rot="MR0">
+<attribute name="POPULARITY" value="3" x="2.91" y="30.25" size="1.778" layer="28" rot="MR0" display="off"/>
 <attribute name="TP_SIGNAL_NAME" value="" x="3.545" y="28.345" size="1" layer="38" rot="MR0"/>
 <attribute name="VALUE" x="3.545" y="29.488" size="0.0254" layer="28" rot="MR0"/>
 <attribute name="VALUE" x="3.545" y="29.488" size="0.0254" layer="28" rot="MR0"/>
 </element>
-<element name="TP3" library="testpad" package="B1,27" value="TPB1,27" x="2.39" y="28.25" smashed="yes" rot="MR0">
+<element name="TP3" library="testpad" library_urn="urn:adsk.eagle:library:385" package="TP10R" package3d_urn="urn:adsk.eagle:package:27959/1" value="TPTP10R" x="2.39" y="28.25" smashed="yes" rot="MR0">
+<attribute name="POPULARITY" value="3" x="2.39" y="28.25" size="1.778" layer="28" rot="MR0" display="off"/>
 <attribute name="TP_SIGNAL_NAME" value="" x="3.025" y="26.345" size="1" layer="38" rot="MR0"/>
 </element>
-<element name="TP4" library="testpad" package="B1,27" value="TPB1,27" x="4.07" y="31.25" smashed="yes" rot="MR0">
+<element name="TP4" library="testpad" library_urn="urn:adsk.eagle:library:385" package="TP10R" package3d_urn="urn:adsk.eagle:package:27959/1" value="TPTP10R" x="4.07" y="31.25" smashed="yes" rot="MR0">
+<attribute name="POPULARITY" value="3" x="4.07" y="31.25" size="1.778" layer="28" rot="MR0" display="off"/>
 <attribute name="TP_SIGNAL_NAME" value="" x="4.705" y="29.345" size="1" layer="38" rot="MR0"/>
 </element>
-<element name="TP5" library="testpad" package="B1,27" value="TPB1,27" x="1.75" y="5.25" smashed="yes" rot="MR0">
+<element name="TP5" library="testpad" library_urn="urn:adsk.eagle:library:385" package="TP10R" package3d_urn="urn:adsk.eagle:package:27959/1" value="TPTP10R" x="1.75" y="5.25" smashed="yes" rot="MR0">
+<attribute name="POPULARITY" value="3" x="1.75" y="5.25" size="1.778" layer="28" rot="MR0" display="off"/>
 <attribute name="TP_SIGNAL_NAME" value="" x="2.385" y="3.345" size="1" layer="38" rot="MR0"/>
 <attribute name="VALUE" x="2.385" y="4.488" size="0.0254" layer="28" rot="MR0"/>
 <attribute name="VALUE" x="2.385" y="4.488" size="0.0254" layer="28" rot="MR0"/>
 </element>
-<element name="TP6" library="testpad" package="B1,27" value="TPB1,27" x="1.63" y="22.25" smashed="yes" rot="MR0">
+<element name="TP6" library="testpad" library_urn="urn:adsk.eagle:library:385" package="TP10R" package3d_urn="urn:adsk.eagle:package:27959/1" value="TPTP10R" x="1.63" y="22.25" smashed="yes" rot="MR0">
+<attribute name="POPULARITY" value="3" x="1.63" y="22.25" size="1.778" layer="28" rot="MR0" display="off"/>
 <attribute name="TP_SIGNAL_NAME" value="" x="2.265" y="20.345" size="1" layer="38" rot="MR0"/>
 <attribute name="VALUE" x="2.265" y="21.488" size="0.0254" layer="28" rot="MR0"/>

Commit message: Improvement and other changes
Parts:
- C3: value (none) -> 100nF
- C6: value (none) -> 10nF
Changed lines of the file:
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@@
 <attribute name="VALUE" x="23.936259375" y="45.46" size="0.4064" layer="27" rot="R270"/>
 </element>
-<element name="C3" library="rcl" package="C0603" value="" x="22" y="20" smashed="yes" rot="MR180">
+<element name="C3" library="rcl" package="C0603" value="100nF" x="22" y="20" smashed="yes" rot="MR180">
 <attribute name="NAME" x="20.965" y="18.965" size="1.27" layer="26" rot="MR180"/>
 <attribute name="VALUE" x="21.365" y="21.905" size="1.27" layer="28" rot="MR180"/>
@@
 <attribute name="VALUE" x="25.768" y="10.511" size="1.27" layer="28" rot="MR90"/>
 </element>
-<element name="C6" library="rcl" package="C0603" value="" x="27.4" y="20.2" smashed="yes" rot="MR270">
+<element name="C6" library="rcl" package="C0603" value="10nF" x="27.4" y="20.2" smashed="yes" rot="MR270">
 <attribute name="NAME" x="29.365" y="21.235" size="1.27" layer="26" rot="MR270"/>
 <attribute name="VALUE" x="29.305" y="20.835" size="1.27" layer="28" rot="MR270"/>

Commit message: Improvement, fixes and other changes
Parts:
- removed U2: ATMEGA328P-MU, Microcontroller:VQFN-32
- added IC4: MEGA8-AI, atmel:TQFP32-08
- moved TP6 17.3 mm to (18.8, 20.1)
- moved TP5 12.4 mm to (14.2, 5.05)
- moved C5 6.55 mm to (7.26, 16.0), turned to 180 degrees
- moved TP1 4.88 mm to (13.2, 22.1)
- moved TP4 3.80 mm to (6.80, 28.6)
- moved TP2 3.03 mm to (3.31, 27.2)
- moved TP3 2.67 mm to (2.99, 30.9)
Connections:
- removed net AREF: U2.20
- removed net N$6: U2.8
- removed net N$8: U2.7
- new net AVCC: IC4.18
- net 5V: now also IC4.4, IC4.6; no longer U2.18, U2.4, U2.6
- net BT0: now also IC4.1; no longer U2.32
- net BT1: now also IC4.32; no longer U2.1
- net GND: now also IC4.21, IC4.3, IC4.5; no longer U2.21, U2.3, U2.33, U2.5
- net LATCH: now also IC4.10; no longer U2.25
- net LEDDATA: now also IC4.13; no longer U2.12
- net MISO: now also IC4.16; no longer U2.16
- net MOSI: now also IC4.15; no longer U2.15
- net PWM: now also IC4.14; no longer U2.13
- net RCLK: now also IC4.11; no longer U2.24
- net RES: now also IC4.29; no longer U2.29
- net RX: now also IC4.30; no longer U2.30
- net SCK: now also IC4.17; no longer U2.17
- net SCL: now also IC4.28; no longer U2.28
- net SDA: now also IC4.27; no longer U2.27
- net SER: now also IC4.9; no longer U2.26
- net TX: now also IC4.31; no longer U2.31
Routing:
- net LATCH: track 56.4 -> 119.2 mm, vias 4 -> 2
- net BT1: track 22.4 -> 85.1 mm, vias 2 -> 5
- net BT0: track 22.7 -> 71.3 mm, vias 0 -> 10
- net GND: track 217.5 -> 183.0 mm, vias 6 -> 4
- net RCLK: track 27.6 -> 47.3 mm, vias 2 -> 4
- net COL5: track 125.1 -> 107.1 mm, vias 15 -> 12
- net 5V: track 133.7 -> 119.3 mm
- net SER: track 13.1 -> 22.5 mm, vias 2 -> 4
- net MOSI: track 1.62 -> 7.18 mm
- net LEDDATA: track 16.0 -> 12.6 mm
- net COL3: track 131.9 -> 128.8 mm
- net PWM: track 59.7 -> 62.6 mm
- net COL0: track 56.8 -> 59.6 mm
- net SCL: track 13.7 -> 16.5 mm
- net COL4: track 58.2 -> 59.6 mm
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