File: tiny-blink-mcu/schematic/tinyblick2.brd (EAGLE design)
At the start: 35 x 35 mm, 51 parts, among them IC3 74LS595D, IC4 74LS595D, J1 USB-MICROB

Commit message: Improvement and other changes
Parts:
- C10: value 10nF -> 100nF
Changed lines of the file:
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@@
 <grid distance="0.1" unitdist="mm" unit="mm" style="lines" multiple="1" display="no" altdistance="5" altunitdist="mil" altunit="mil"/>
 <layers>
-<layer number="1" name="Top" color="4" fill="1" visible="no" active="yes"/>
+<layer number="1" name="Top" color="4" fill="1" visible="yes" active="yes"/>
 <layer number="16" name="Bottom" color="1" fill="1" visible="yes" active="yes"/>
 <layer number="17" name="Pads" color="2" fill="1" visible="yes" active="yes"/>
@@
 <layer number="19" name="Unrouted" color="6" fill="1" visible="yes" active="yes"/>
 <layer number="20" name="Dimension" color="15" fill="1" visible="yes" active="yes"/>
-<layer number="21" name="tPlace" color="7" fill="1" visible="no" active="yes"/>
+<layer number="21" name="tPlace" color="7" fill="1" visible="yes" active="yes"/>
 <layer number="22" name="bPlace" color="7" fill="1" visible="yes" active="yes"/>
-<layer number="23" name="tOrigins" color="15" fill="1" visible="no" active="yes"/>
+<layer number="23" name="tOrigins" color="15" fill="1" visible="yes" active="yes"/>
 <layer number="24" name="bOrigins" color="15" fill="1" visible="yes" active="yes"/>
-<layer number="25" name="tNames" color="7" fill="1" visible="no" active="yes"/>
+<layer number="25" name="tNames" color="7" fill="1" visible="yes" active="yes"/>
 <layer number="26" name="bNames" color="7" fill="1" visible="yes" active="yes"/>
 <layer number="27" name="tValues" color="7" fill="1" visible="no" active="yes"/>
@@
 <layer number="37" name="tTest" color="7" fill="1" visible="no" active="yes"/>
 <layer number="38" name="bTest" color="7" fill="1" visible="no" active="yes"/>
-<layer number="39" name="tKeepout" color="4" fill="11" visible="no" active="yes"/>
+<layer number="39" name="tKeepout" color="4" fill="11" visible="yes" active="yes"/>
 <layer number="40" name="bKeepout" color="1" fill="11" visible="yes" active="yes"/>
-<layer number="41" name="tRestrict" color="4" fill="10" visible="no" active="yes"/>
+<layer number="41" name="tRestrict" color="4" fill="10" visible="yes" active="yes"/>
 <layer number="42" name="bRestrict" color="1" fill="10" visible="yes" active="yes"/>
 <layer number="43" name="vRestrict" color="2" fill="10" visible="no" active="yes"/>
@@
 <layer number="49" name="Reference" color="7" fill="1" visible="no" active="yes"/>
 <layer number="50" name="dxf" color="7" fill="1" visible="no" active="no"/>
-<layer number="51" name="tDocu" color="7" fill="1" visible="no" active="yes"/>
+<layer number="51" name="tDocu" color="7" fill="1" visible="yes" active="yes"/>
 <layer number="52" name="bDocu" color="7" fill="1" visible="yes" active="yes"/>
 <layer number="53" name="tGND_GNDA" color="7" fill="9" visible="no" active="no"/>
@@
 <attribute name="VALUE" x="18.335003125" y="28.97" size="0.4064" layer="28" rot="MR270"/>
 </element>
-<element name="C10" library="adafruit" package="C0603" value="10nF" x="17.8" y="31.3" smashed="yes" rot="MR180">
+<element name="C10" library="adafruit" package="C0603" value="100nF" x="17.8" y="31.3" smashed="yes" rot="MR180">
 <attribute name="NAME" x="16.111" y="33.438" size="1.27" layer="26" rot="MR180"/>
 <attribute name="VALUE" x="16.911" y="33.332" size="1.27" layer="28" rot="MR180"/>
@@
 <wire x1="12.4211375" y1="16.6682" x2="14.84805625" y2="16.6682" width="0.1524" layer="1"/>
 <wire x1="14.84805625" y1="16.6682" x2="15.595" y2="17.41514375" width="0.1524" layer="1"/>
-<via x="14.8302" y="22.5" extent="1-16" drill="0.35"/>
+<via x="14.8302" y="22.5" extent="1-16" drill="0.3"/>
 <wire x1="14.8302" y1="22.5" x2="14.8" y2="22.5" width="0.1524" layer="16"/>
 <wire x1="14.8302" y1="22.5" x2="13.4" y2="22.5" width="0.1524" layer="16"/>
 <wire x1="13.4" y1="22.5" x2="11.9" y2="21" width="0.1524" layer="16"/>
 <wire x1="11.9" y1="21" x2="11.94466875" y2="21" width="0.1524" layer="16"/>
-<via x="11.94466875" y="21" extent="1-16" drill="0.35"/>
+<via x="11.94466875" y="21" extent="1-16" drill="0.3"/>
 <wire x1="14.8302" y1="22.5" x2="14.8302" y2="27.9198" width="0.1524" layer="1"/>
 <wire x1="14.8302" y1="27.9198" x2="13.75" y2="29" width="0.1524" layer="1"/>
@@
 <wire x1="15.0838" y1="25.795" x2="15.125" y2="25.7538" width="0.2032" layer="16"/>
 <wire x1="15.125" y1="25.7538" x2="15.125" y2="23.25" width="0.2032" layer="16"/>
-<wire x1="15.125" y1="23.25" x2="15.125" y2="23.175" width="0.2032" layer="16"/>
-<wire x1="15.125" y1="23.175" x2="16.9" y2="21.4" width="0.2032" layer="16"/>
+<wire x1="15.125" y1="23.25" x2="15.125" y2="23.075" width="0.2032" layer="16"/>
+<wire x1="16.8" y1="21.4" x2="16.9" y2="21.4" width="0.2032" layer="16"/>
+<wire x1="16.8" y1="21.4" x2="15.125" y2="23.075" width="0.2032" layer="16"/>
 <wire x1="17.1" y1="21.4" x2="16.9" y2="21.4" width="0.2032" layer="16"/>
 <wire x1="14.7" y1="25.8" x2="14.8875" y2="25.9875" width="0.2032" layer="16"/>
@@
 <wire x1="17.225" y1="27.625" x2="16.425" y2="27.625" width="0.1524" layer="16"/>
 <wire x1="16.3" y1="27.75" x2="16.425" y2="27.625" width="0.1524" layer="16"/>
-<wire x1="9.8382" y1="29.3382" x2="11.9118" y2="29.3382" width="0.1524" layer="16"/>
+<wire x1="9.9382" y1="29.3382" x2="11.9118" y2="29.3382" width="0.1524" layer="16"/>
 <wire x1="11.9118" y1="29.3382" x2="13.5" y2="27.75" width="0.1524" layer="16"/>
 <wire x1="13.5" y1="27.75" x2="16.3" y2="27.75" width="0.1524" layer="16"/>
-<wire x1="9.8382" y1="29.2382" x2="9.8382" y2="29.3382" width="0.1524" layer="16"/>
-<wire x1="6.5" y1="25.9" x2="9.8382" y2="29.2382" width="0.1524" layer="16"/>
+<wire x1="6.5" y1="25.9" x2="9.9382" y2="29.3382" width="0.1524" layer="16"/>
 </signal>
 <signal name="N$2">
