File: christmascard/schematic/christmas_card.sch (EAGLE design)
At the start: 74 parts, among them IC1 WS2811-SOP8, IC2 WS2811-SOP8, IC5 WS2811-SOP8, IC7 74LS595D, U3 ATTINY24/44/84-SSU, X2 USB-MICROB

Commit message: Improvement, fixes and other changes
Connections:
- removed net LEDATA: U3.(PCINT0/AREF/ADC0)PA0
- net LEDDATA: now also U3.(PCINT0/AREF/ADC0)PA0
Changed lines of the file:
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@@
 <label x="457.2" y="162.56" size="1.778" layer="95" rot="R270" xref="yes"/>
+</segment>
+<segment>
+<pinref part="U3" gate="&gt;NAME" pin="(PCINT0/AREF/ADC0)PA0"/>
+<wire x1="558.8" y1="111.76" x2="574.04" y2="111.76" width="0.1524" layer="91"/>
+<label x="574.04" y="111.76" size="1.778" layer="95" xref="yes"/>
 </segment>
 </net>
@@
 </segment>
 </net>
-<net name="LEDATA" class="0">
-<segment>
-<pinref part="U3" gate="&gt;NAME" pin="(PCINT0/AREF/ADC0)PA0"/>
-<wire x1="558.8" y1="111.76" x2="574.04" y2="111.76" width="0.1524" layer="91"/>
-<label x="574.04" y="111.76" size="1.778" layer="95" xref="yes"/>
-</segment>
-</net>
